File: hardware/ReflowController_true_rev2.sch (EAGLE design)
At the start: 45 parts, among them IC1 MAX31855, IC2 MAX31855

Commit message: Board: Fixed C7 mains cap size
Changed C7 cap to a standard 15mm width X2 cap. Reworked the board in
this area to get it to fit.
Parts:
- C7: device rcl:C-EU025-025X050 -> rcl:C-EU150-054X183
Connections:
- removed net N$10: C7.2, OC1.C, R10.2
- new net N$6: C7.2, OC1.A, R9.2
- net N$9: now also OC1.C, R10.2; no longer OC1.A, R9.2
Other:
- moved on the sheet: C7
Changed lines of the file:
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@@
 <setting verticaltext="up"/>
 </settings>
-<grid distance="0.1" unitdist="inch" unit="inch" style="lines" multiple="1" display="yes" altdistance="0.01" altunitdist="inch" altunit="inch"/>
+<grid distance="0.1" unitdist="inch" unit="inch" style="lines" multiple="1" display="no" altdistance="0.01" altunitdist="inch" altunit="inch"/>
 <layers>
 <layer number="1" name="Top" color="4" fill="1" visible="no" active="no"/>
@@
 <part name="C5" library="rcl" deviceset="C-EU" device="C0805" value="10n"/>
 <part name="GND10" library="supply1" deviceset="GND" device=""/>
-<part name="C7" library="rcl" deviceset="C-EU" device="025-025X050" value="100n"/>
+<part name="C7" library="rcl" deviceset="C-EU" device="150-054X183" value="100n"/>
 <part name="GND11" library="supply1" deviceset="GND" device=""/>
 <part name="OC1" library="optocoupler" deviceset="PC817" device=""/>
@@
 </instance>
 <instance part="GND10" gate="1" x="10.16" y="180.34" smashed="yes"/>
-<instance part="C7" gate="G$1" x="45.72" y="109.22" smashed="yes">
-<attribute name="NAME" x="44.704" y="113.919" size="1.778" layer="95"/>
-<attribute name="VALUE" x="43.434" y="100.965" size="1.778" layer="96"/>
+<instance part="C7" gate="G$1" x="45.72" y="106.68" smashed="yes" rot="R180">
+<attribute name="NAME" x="46.736" y="101.981" size="1.778" layer="95" rot="R180"/>
+<attribute name="VALUE" x="48.006" y="114.935" size="1.778" layer="96" rot="R180"/>
 </instance>
 <instance part="GND11" gate="1" x="55.88" y="144.78" smashed="yes"/>
@@
 </segment>
 </net>
-<net name="N$9" class="0">
-<segment>
-<pinref part="R9" gate="G$1" pin="2"/>
-<pinref part="C7" gate="G$1" pin="1"/>
-<wire x1="45.72" y1="111.76" x2="48.26" y2="111.76" width="0.1524" layer="91"/>
-<pinref part="OC1" gate="A" pin="A"/>
-<wire x1="38.1" y1="109.22" x2="40.64" y2="109.22" width="0.1524" layer="91"/>
-<wire x1="40.64" y1="109.22" x2="40.64" y2="111.76" width="0.1524" layer="91"/>
-<wire x1="40.64" y1="111.76" x2="45.72" y2="111.76" width="0.1524" layer="91"/>
-<junction x="45.72" y="111.76"/>
-</segment>
-</net>
-<net name="N$10" class="0">
-<segment>
-<pinref part="R10" gate="G$1" pin="2"/>
-<pinref part="C7" gate="G$1" pin="2"/>
-<wire x1="45.72" y1="104.14" x2="48.26" y2="104.14" width="0.1524" layer="91"/>
-<pinref part="OC1" gate="A" pin="C"/>
-<wire x1="38.1" y1="104.14" x2="45.72" y2="104.14" width="0.1524" layer="91"/>
-<junction x="45.72" y="104.14"/>
-</segment>
-</net>
 <net name="ZEROX" class="0">
 <segment>
@@
 </segment>
 </net>
+<net name="N$6" class="0">
+<segment>
+<wire x1="40.64" y1="109.22" x2="40.64" y2="111.76" width="0.1524" layer="91"/>
+<pinref part="OC1" gate="A" pin="A"/>
+<wire x1="38.1" y1="109.22" x2="40.64" y2="109.22" width="0.1524" layer="91"/>
+<pinref part="R9" gate="G$1" pin="2"/>
+<pinref part="C7" gate="G$1" pin="2"/>
+<wire x1="48.26" y1="111.76" x2="45.72" y2="111.76" width="0.1524" layer="91"/>
+<wire x1="45.72" y1="111.76" x2="40.64" y2="111.76" width="0.1524" layer="91"/>
+<junction x="45.72" y="111.76"/>
+</segment>
+</net>
+<net name="N$9" class="0">
+<segment>
+<pinref part="R10" gate="G$1" pin="2"/>
+<pinref part="C7" gate="G$1" pin="1"/>
+<wire x1="48.26" y1="104.14" x2="45.72" y2="104.14" width="0.1524" layer="91"/>
+<pinref part="OC1" gate="A" pin="C"/>
+<wire x1="45.72" y1="104.14" x2="38.1" y2="104.14" width="0.1524" layer="91"/>
+<junction x="45.72" y="104.14"/>
+</segment>
+</net>
